File: mini-power/mini-power.kicad_sch (KiCad schematic)
At the start: 0 parts

Commit message: Add power supply schematic, parts libraries and design docs
- Schematic (A2, generated by tools/gen_schematic.py): +2.8 V and +1.4 V
  TPS6284x bucks, -2.8 V LT8330 inverter, and controller-driven +1.375 V
  buck and -2.75 V inverter options (charge pump / P-FET + inductor) with
  an LPV521 sense amplifier, series current jumpers and one test point per net
- LCSC parts imported with easyeda2kicad into mini-power/lib
- Design notes and calculations in docs/, project rules in CLAUDE.md

Co-Authored-By: Claude Sonnet 5.5 <noreply@anthropic.com>
Parts:
- added C1, C10, C12, C13, C3, C5: 4.7uF/10V, mp:C0402, symbol mp:CL05A475MP5NRNC
- added C11, C6, C9: 1uF/50V, mp:C0603, symbol mp:CL10A105KB8NNNC
- added C14: 100nF, mp:C0402, symbol mp:CL05B104KO5NNNC
- added C15: 10pF, mp:C0402, symbol mp:CC0402JRNPO9BN100
- added C2, C4, C7: 10uF/6.3V, mp:C0402, symbol mp:CGA0402X5R106M6R3GT
- added C8: 4.7pF, mp:C0402, symbol mp:0402CG4R7C500NT
- added D1, D2, D3, D4: PMEG6010CEJ, mp:SOD-323F_L2.0-W1.6-LS2.5-RD, symbol mp:PMEG6010CEJ,115
- added J1: Power in, mp:HDR-TH_2P-P2.54-V-M, symbol mp:PZ254V-11-02P
- added J2: Power out, mp:HDR-TH_4P-P2.54-V-M, symbol mp:PZ254V-11-04P_C2691448
- added J3: +2.75 V in, mp:HDR-TH_2P-P2.54-V-M, symbol mp:PZ254V-11-02P
- added J4: Controller rails out, mp:HDR-TH_3P-P2.54-V-M_PZ254V-11-03P, symbol mp:PZ254V-11-03P_C2937625
- added J5: Controller, mp:HDR-TH_6P-P2.54-V-M, symbol mp:PZ254V-11-06P
- added JP1, JP2, JP3, JP4: Current jumper, mp:HDR-TH_2P-P2.54-V-M, symbol mp:PZ254V-11-02P
- added JP5: Current jumper A, mp:HDR-TH_2P-P2.54-V-M, symbol mp:PZ254V-11-02P
- added JP6: Current jumper B, mp:HDR-TH_2P-P2.54-V-M, symbol mp:PZ254V-11-02P
- added L1, L2, L3, L4: 2.2uH, mp:L0806, symbol mp:DFE201612E-2R2M=P2
- added L5: 100uH, mp:L0805, symbol mp:LBR2012T101M
- added L6: 47uH, mp:L0805, symbol mp:LB2012T470M
- added Q1: Si2301CDS, mp:SOT-23-3_L3.0-W1.7-P0.95-LS2.9-BR, symbol mp:SI2301CDS-T1-GE3
- added R1: 28.7k 1%, mp:R0402, symbol mp:0402WGF2872TCE
- added R2: 52.3k 1%, mp:R0402, symbol mp:0402WGF5232TCE
- added R3, R5: 1M 1%, mp:R0402, symbol mp:0402WGF1004TCE
- added R4: 402k 1%, mp:R0402, symbol mp:0402WGF4023TCE
- added R6: 4.99M 1%, mp:R0402, symbol mp:RC0402FR-074M99L
- added R7: 2.49M 1%, mp:R0402, symbol mp:FRC0402F2494TS
- added TP1: SW_A, mp:TestPoint_0.5mm, symbol mpx:TestPoint
- added TP10: CPL_C, mp:TestPoint_0.5mm, symbol mpx:TestPoint
- added TP11: FBX_C, mp:TestPoint_0.5mm, symbol mpx:TestPoint
- added TP12: INTVCC_C, mp:TestPoint_0.5mm, symbol mpx:TestPoint
- added TP13: -2V8_IC, mp:TestPoint_0.5mm, symbol mpx:TestPoint
- added TP14: -2V8, mp:TestPoint_0.5mm, symbol mpx:TestPoint
- added TP15: +3V3, mp:TestPoint_0.5mm, symbol mpx:TestPoint
- added TP16: GND, mp:TestPoint_0.5mm, symbol mpx:TestPoint
- added TP17: +2V75, mp:TestPoint_0.5mm, symbol mpx:TestPoint
- added TP18: BUCK_DRV, mp:TestPoint_0.5mm, symbol mpx:TestPoint
- added TP19: +1V375_IC, mp:TestPoint_0.5mm, symbol mpx:TestPoint
- added TP2: VSET_A, mp:TestPoint_0.5mm, symbol mpx:TestPoint
- added TP20: +1V375, mp:TestPoint_0.5mm, symbol mpx:TestPoint
- added TP21: A_DRV, mp:TestPoint_0.5mm, symbol mpx:TestPoint
- added TP22: N_A, mp:TestPoint_0.5mm, symbol mpx:TestPoint
- added TP23: -2V75_A, mp:TestPoint_0.5mm, symbol mpx:TestPoint
- added TP24: B_DRV, mp:TestPoint_0.5mm, symbol mpx:TestPoint
- added TP25: SW_PB, mp:TestPoint_0.5mm, symbol mpx:TestPoint
- added TP26: -2V75_B, mp:TestPoint_0.5mm, symbol mpx:TestPoint
- added TP27: SNS_IN, mp:TestPoint_0.5mm, symbol mpx:TestPoint
- added TP28: SENSE, mp:TestPoint_0.5mm, symbol mpx:TestPoint
- added TP29: -2V75, mp:TestPoint_0.5mm, symbol mpx:TestPoint
- added TP3: +2V8_IC, mp:TestPoint_0.5mm, symbol mpx:TestPoint
- added TP4: +2V8, mp:TestPoint_0.5mm, symbol mpx:TestPoint
- added TP5: SW_B, mp:TestPoint_0.5mm, symbol mpx:TestPoint
- added TP6: VSET_B, mp:TestPoint_0.5mm, symbol mpx:TestPoint
- added TP7: +1V4_IC, mp:TestPoint_0.5mm, symbol mpx:TestPoint
- added TP8: +1V4, mp:TestPoint_0.5mm, symbol mpx:TestPoint
- added TP9: SW_C, mp:TestPoint_0.5mm, symbol mpx:TestPoint
- added U1: TPS62840DLC, mp:VSON-8_L2.0-W1.5-P0.50-BL, symbol mp:TPS62840DLCR
- added U2: TPS62841DLC, mp:VSON-8_L2.0-W1.5-P0.50-BL, symbol mp:TPS62841DLCR
- added U3: LT8330, mp:SOT-23-6_L2.9-W1.6-P0.95-LS2.8-BR, symbol mp:LT8330ES6#TRMPBF
- added U4: LPV521, mp:SC-70-5_L2.0-W1.3-P0.65-LS2.2-BL, symbol mp:LPV521MGX_NOPB
Connections:
- new net +1V375: J4.2, JP4.2, TP20.1
- new net +1V375_IC: C10.2, JP4.1, L5.2, TP19.1
- new net +1V4: J2.4, JP2.2, TP8.1
- new net +1V4_IC: C4.2, JP2.1, L2.2, TP7.1, U2.8 (VOS)
- new net +2V75: C14.2, J3.1, J5.1, Q1.2 (S), R5.2, TP17.1, U4.5 (V+)
- new net +2V8: J2.2, JP1.2, TP4.1
- new net +2V8_IC: C2.2, JP1.1, L1.2, TP3.1, U1.8 (VOS)
- new net +3V3: C1.2, C3.2, C5.2, J1.1, L3.1, TP15.1, U1.2 (VIN), U1.4 (EN), U2.2 (VIN), U2.4 (EN), U3.4 (EN/UVLO), U3.6 (VIN)
- new net -2V75: J4.3, JP5.2, JP6.2, TP29.1
- new net -2V75_A: C12.2, D3.2 (A), JP5.1, TP23.1
- new net -2V75_B: C13.2, D4.2 (A), JP6.1, R6.1, TP26.1
- new net -2V8: J2.3, JP3.2, TP14.1
- new net -2V8_IC: C7.2, C8.2, JP3.1, L4.2, R3.2, TP13.1
- new net A_DRV: C11.1, J5.4, TP21.1
- new net BUCK_DRV: J5.3, L5.1, TP18.1
- new net B_DRV: J5.5, Q1.1 (G), R5.1, TP24.1
- new net CPL_C: C6.2, D1.2 (A), L4.1, TP10.1
- new net FBX_C: C8.1, R3.1, R4.2, TP11.1, U3.3 (FBX)
- new net GND: C1.1, C10.1, C12.1, C13.1, C14.1, C2.1, C3.1, C4.1, C5.1, C7.1, C9.1, D1.1 (C), D2.1 (C), J1.2, J2.1, J3.2, J4.1, J5.2, L6.1, R1.1, R2.1, R4.1, TP16.1, U1.1 (GND), U1.3 (MODE), U1.6 (STOP), U2.1 (GND), U2.3 (MODE), U2.6 (STOP), U3.2 (GND), U4.2 (V-), U4.3 (IN+)
- new net INTVCC_C: C9.2, TP12.1, U3.5 (INTVCC)
- new net N_A: C11.2, D2.2 (A), D3.1 (C), TP22.1
- new net SENSE: C15.2, J5.6, R7.2, TP28.1, U4.1 (OUT)
- new net SNS_IN: C15.1, R6.2, R7.1, TP27.1, U4.4 (IN-)
- new net SW_A: L1.1, TP1.1, U1.7 (SW)
- new net SW_B: L2.1, TP5.1, U2.7 (SW)
- new net SW_C: C6.1, L3.2, TP9.1, U3.1 (SW)
- new net SW_PB: D4.1 (C), L6.2, Q1.3 (D), TP25.1
- new net VSET_A: R1.2, TP2.1, U1.5 (VSET)
- new net VSET_B: R2.2, TP6.1, U2.5 (VSET)
Other:
- note added: "-2.75 V output jumpers (fit only ONE)"
- note added: "3.3 V -> 1.4 V, 5 mA max. MODE = GND: auto PFM, 60 nA Iq. Output passes JP2 (jumper or ammeter)."
- note added: "3.3 V -> 2.8 V, 5 mA max. MODE = GND: auto PFM, 60 nA Iq. Output passes JP1 (jumper or ammeter)."
- note added: "A_DRV swings the flying capacitor 0 to 2.75 V; D2 and D3 steer the charge. Unregulated output about -2.1 to -2.4 V (cannot reach -2.75 V)."
- note added: "BUCK_DRV is a push-pull timer output (about 2 MHz, duty 0.516). L5 and the output capacitor filter it; the pin sinks current too,"
- note added: "B_DRV gates Q1 (low = on). While Q1 is on, L6 charges from +2.75 V; when it turns off the stored energy flows through D4 into the negative rail."
- note added: "Block A: +2.8 V buck (U1 TPS62840, RSET 28.7k selects 2.8 V)"
- note added: "Block B: +1.4 V buck (U2 TPS62841, RSET 52.3k selects 1.4 V)"
- note added: "Block C: -2.8 V inverting converter (U3 LT8330, dual-inductor topology)"
- note added: "Block D: +1.375 V buck, inductor driven directly from a controller pin"
- note added: "Block E-A: -2.75 V inverter, option A (pin-driven charge pump, no inductor)"
- note added: "Block E-B: -2.75 V inverter, option B (P-FET + inductor, regulated by the controller in burst mode)"
- note added: "Controller interface"
- note added: "Controller-driven rails (separate +2.75 V supply, generic low-power STM32 on J5)"
- note added: "Design notes, assumptions and the unregulated load swing: docs/controller-rails.md"
- note added: "Generic low-power STM32. Pin 1 powers it from +2.75 V. Pins 3 to 5: timer outputs. Pin 6: analog input (sense)."
- note added: "Input"
- note added: "Input +2.75 V"
- note added: "JP5: charge pump (option A) JP6: inductor stage (option B)"
- note added: "L3/L4, CDC and D1 form the inverting stage. The divider R3/R4 sets VOUT = -0.8 V x (1 + R3/R4) = -2.79 V. EN/UVLO is tied to +3V3."
- note added: "Outputs"
- note added: "Outputs (controller rails)"
- note added: "Pin 1: +2.75 V Pin 2: GND"
- note added: "Pin 1: +3.3 V Pin 2: GND"
- note added: "Pin 1: GND Pin 2: +1.375 V Pin 3: -2.75 V"
- note added: "Pin 1: GND Pin 2: +2.8 V Pin 3: -2.8 V Pin 4: +1.4 V"
- note added: "U4 (LPV521, 0.35 uA) inverts the rail into SENSE = 0.499 x |VRAIL| (1.37 V at -2.75 V); the controller skips pulses once SENSE reaches the target."
- note added: "VIN must stay above 3.0 V (LT8330 minimum). SW swings between 0 V and VIN + |VOUT| = 6.1 V. Output passes JP3."
- note added: "so the stage stays in continuous conduction at any load and the unregulated output follows the load only by the pin resistance."
- title: (none) -> Mini-power

Commit message: Add switching frequency and duty cycle for all converters
- Schematic notes under every block: TPS62840/41 and LT8330 (integrated)
  and the three controller-driven stages (pin buck, charge pump, P-FET stage)
- docs/power-architecture.md section 8 and docs/controller-rails.md section 8.4
- tools/integrated_rails_model.py reproduces the integrated-rail estimates

Co-Authored-By: Claude Sonnet 5.5 <noreply@anthropic.com>
Other:
- note added: "A_DRV: f = 500 kHz (100 kHz to 1 MHz works), duty D = 0.50 (symmetric square wave)."
- note added: "BUCK_DRV: f = 2 MHz, duty D = 0.516 for 1.375 V at 1 mA (0.5016 at 0.1 mA, 0.532 at 2 mA; ideal 1.375 / 2.75 = 0.500). Needs a timer clock of 64 MHz or more for steps below 90 mV."
- note added: "B_DRV: fixed ton = 0.855 us (Ipk 50 mA in L6), toff 0.80 us; burst rate 6 / 61 / 122 kHz = average duty 0.5 / 5.2 / 10.4 % for 0.1 / 1 / 2 mA."
- note added: "Switching: 1.8 MHz nominal (PWM), duty D = 1.4 / 3.3 = 0.424 (ton 236 ns). At 0.1 / 1 / 5 mA it runs in power-save (PFM) at about 2 / 18 / 88 kHz (estimate)."
- note added: "Switching: 1.8 MHz nominal (PWM), duty D = 2.8 / 3.3 = 0.848 (ton 471 ns). At 0.1 / 1 / 5 mA it runs in power-save (PFM) at about 3 / 34 / 168 kHz (estimate)."
- note added: "Switching: fixed 2 MHz oscillator (CCM duty D = (2.79 + 0.3) / (2.79 + 0.3 + 3.3) = 0.484, ton 242 ns); below about 17 mA it runs in Burst Mode:"
- note added: "single pulses (ton about 80 ns, 240 mA switch limit) at about 11 / 114 / 572 kHz for 0.1 / 1 / 5 mA (estimate)."
Changed lines of the file:
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@@
 	(text "Block A: +2.8 V buck (U1 TPS62840, RSET 28.7k selects 2.8 V)" (exclude_from_sim no) (at 83.82 33.02 0) (effects (font (size 2.0 2.0) bold) (justify left top)))
 	(text "3.3 V -> 2.8 V, 5 mA max. MODE = GND: auto PFM, 60 nA Iq. Output passes JP1 (jumper or ammeter)." (exclude_from_sim no) (at 83.82 38.1 0) (effects (font (size 1.27 1.27)) (justify left top)))
+	(text "Switching: 1.8 MHz nominal (PWM), duty D = 2.8 / 3.3 = 0.848 (ton 471 ns). At 0.1 / 1 / 5 mA it runs in power-save (PFM) at about 3 / 34 / 168 kHz (estimate)." (exclude_from_sim no) (at 83.82 41.91 0) (effects (font (size 1.27 1.27)) (justify left top)))
 	(wire (pts (xy 102.87 59.69) (xy 100.33 59.69)) (stroke (width 0) (type default)))
 	(label "GND" (at 100.33 59.69 0) (effects (font (size 1.27 1.27)) (justify right bottom)))
@@
 	(text "Block B: +1.4 V buck (U2 TPS62841, RSET 52.3k selects 1.4 V)" (exclude_from_sim no) (at 83.82 109.22 0) (effects (font (size 2.0 2.0) bold) (justify left top)))
 	(text "3.3 V -> 1.4 V, 5 mA max. MODE = GND: auto PFM, 60 nA Iq. Output passes JP2 (jumper or ammeter)." (exclude_from_sim no) (at 83.82 114.3 0) (effects (font (size 1.27 1.27)) (justify left top)))
+	(text "Switching: 1.8 MHz nominal (PWM), duty D = 1.4 / 3.3 = 0.424 (ton 236 ns). At 0.1 / 1 / 5 mA it runs in power-save (PFM) at about 2 / 18 / 88 kHz (estimate)." (exclude_from_sim no) (at 83.82 118.11 0) (effects (font (size 1.27 1.27)) (justify left top)))
 	(wire (pts (xy 102.87 135.89) (xy 100.33 135.89)) (stroke (width 0) (type default)))
 	(label "GND" (at 100.33 135.89 0) (effects (font (size 1.27 1.27)) (justify right bottom)))
@@
 	(wire (pts (xy 194.31 140.97) (xy 194.31 143.51)) (stroke (width 0) (type default)))
 	(junction (at 194.31 140.97) (diameter 0) (color 0 0 0 0))
-	(text "Block C: -2.8 V inverting converter (U3 LT8330, dual-inductor topology)" (exclude_from_sim no) (at 73.66 198.12 0) (effects (font (size 2.0 2.0) bold) (justify left top)))
-	(text "L3/L4, CDC and D1 form the inverting stage. The divider R3/R4 sets VOUT = -0.8 V x (1 + R3/R4) = -2.79 V. EN/UVLO is tied to +3V3." (exclude_from_sim no) (at 73.66 203.2 0) (effects (font (size 1.27 1.27)) (justify left top)))
-	(text "VIN must stay above 3.0 V (LT8330 minimum). SW swings between 0 V and VIN + |VOUT| = 6.1 V. Output passes JP3." (exclude_from_sim no) (at 73.66 207.01 0) (effects (font (size 1.27 1.27)) (justify left top)))
+	(text "Block C: -2.8 V inverting converter (U3 LT8330, dual-inductor topology)" (exclude_from_sim no) (at 73.66 191.77 0) (effects (font (size 2.0 2.0) bold) (justify left top)))
+	(text "L3/L4, CDC and D1 form the inverting stage. The divider R3/R4 sets VOUT = -0.8 V x (1 + R3/R4) = -2.79 V. EN/UVLO is tied to +3V3." (exclude_from_sim no) (at 73.66 196.85 0) (effects (font (size 1.27 1.27)) (justify left top)))
+	(text "VIN must stay above 3.0 V (LT8330 minimum). SW swings between 0 V and VIN + |VOUT| = 6.1 V. Output passes JP3." (exclude_from_sim no) (at 73.66 200.66 0) (effects (font (size 1.27 1.27)) (justify left top)))
+	(text "Switching: fixed 2 MHz oscillator (CCM duty D = (2.79 + 0.3) / (2.79 + 0.3 + 3.3) = 0.484, ton 242 ns); below about 17 mA it runs in Burst Mode:" (exclude_from_sim no) (at 73.66 204.47 0) (effects (font (size 1.27 1.27)) (justify left top)))
+	(text "single pulses (ton about 80 ns, 240 mA switch limit) at about 11 / 114 / 572 kHz for 0.1 / 1 / 5 mA (estimate)." (exclude_from_sim no) (at 73.66 208.28 0) (effects (font (size 1.27 1.27)) (justify left top)))
 	(symbol
 		(lib_id "mp:LT8330ES6#TRMPBF")
@@
 	(text "BUCK_DRV is a push-pull timer output (about 2 MHz, duty 0.516). L5 and the output capacitor filter it; the pin sinks current too," (exclude_from_sim no) (at 391.16 43.18 0) (effects (font (size 1.27 1.27)) (justify left top)))
 	(text "so the stage stays in continuous conduction at any load and the unregulated output follows the load only by the pin resistance." (exclude_from_sim no) (at 391.16 46.99 0) (effects (font (size 1.27 1.27)) (justify left top)))
+	(text "BUCK_DRV: f = 2 MHz, duty D = 0.516 for 1.375 V at 1 mA (0.5016 at 0.1 mA, 0.532 at 2 mA; ideal 1.375 / 2.75 = 0.500). Needs a timer clock of 64 MHz or more for steps below 90 mV." (exclude_from_sim no) (at 391.16 50.8 0) (effects (font (size 1.27 1.27)) (justify left top)))
 	(label "BUCK_DRV" (at 391.16 63.5 0) (effects (font (size 1.27 1.27)) (justify left bottom)))
 	(symbol
@@
 	(text "Block E-A: -2.75 V inverter, option A (pin-driven charge pump, no inductor)" (exclude_from_sim no) (at 391.16 104.14 0) (effects (font (size 2.0 2.0) bold) (justify left top)))
 	(text "A_DRV swings the flying capacitor 0 to 2.75 V; D2 and D3 steer the charge. Unregulated output about -2.1 to -2.4 V (cannot reach -2.75 V)." (exclude_from_sim no) (at 391.16 109.22 0) (effects (font (size 1.27 1.27)) (justify left top)))
+	(text "A_DRV: f = 500 kHz (100 kHz to 1 MHz works), duty D = 0.50 (symmetric square wave)." (exclude_from_sim no) (at 391.16 113.03 0) (effects (font (size 1.27 1.27)) (justify left top)))
 	(label "A_DRV" (at 391.16 129.54 0) (effects (font (size 1.27 1.27)) (justify left bottom)))
 	(symbol
@@
 	(text "B_DRV gates Q1 (low = on). While Q1 is on, L6 charges from +2.75 V; when it turns off the stored energy flows through D4 into the negative rail." (exclude_from_sim no) (at 391.16 179.07 0) (effects (font (size 1.27 1.27)) (justify left top)))
 	(text "U4 (LPV521, 0.35 uA) inverts the rail into SENSE = 0.499 x |VRAIL| (1.37 V at -2.75 V); the controller skips pulses once SENSE reaches the target." (exclude_from_sim no) (at 391.16 182.88 0) (effects (font (size 1.27 1.27)) (justify left top)))
+	(text "B_DRV: fixed ton = 0.855 us (Ipk 50 mA in L6), toff 0.80 us; burst rate 6 / 61 / 122 kHz = average duty 0.5 / 5.2 / 10.4 % for 0.1 / 1 / 2 mA." (exclude_from_sim no) (at 391.16 186.69 0) (effects (font (size 1.27 1.27)) (justify left top)))
 	(label "B_DRV" (at 391.16 214.63 0) (effects (font (size 1.27 1.27)) (justify left bottom)))
 	(symbol
