File: mini-power/mini-power.kicad_sch (KiCad schematic)
At the start: 77 parts, among them J1 Power in, J2 Power out, J3 +2.75 V in, J4 Controller rails out, J5 Controller, Q1 Si2301CDS, U1 TPS62840DLC, U2 TPS62841DLC, U3 LT8330, U4 LPV521

Commit message: Corrected PCB layout
Parts:
- removed C11, C6, C9: 1uF/50V, mp:C0603, symbol mp:CL10A105KB8NNNC
- added C11, C6, C9: 1uF/25V, mp:C0402, symbol mp:CL05A105KA5NQNC
Connections:
- net A_DRV: now also C11.1
- net CPL_C: now also C6.2
- net GND: now also C9.1
- net INTVCC_C: now also C9.2
- net N_A: now also C11.2
- net SW_C: now also C6.1
Changed lines of the file:
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@@
 	(label "SW_C" (at 127 233.68 0) (effects (font (size 1.27 1.27)) (justify left bottom)))
 	(symbol
-		(lib_id "mp:CL10A105KB8NNNC")
+		(lib_id "mp:CL05A105KA5NQNC")
 		(at 139.7 215.9 0)
 		(unit 1)
@@
 		(dnp no)
 		(property "Reference" "C6" (at 139.7 212.09 0) (effects (font (size 1.27 1.27))))
-		(property "Value" "1uF/50V" (at 139.7 219.71 0) (effects (font (size 1.27 1.27))))
-		(property "Footprint" "mp:C0603" (at 139.7 215.9 0) (effects (font (size 1.27 1.27)) (hide yes)))
-		(property "Datasheet" "https://lcsc.com/product-detail/Multilayer-Ceramic-Capacitors-MLCC-SMD-SMT_SAMSUNG_CL10A105KB8NNNC_1uF-105-10-50V_C15849.html" (at 139.7 215.9 0) (effects (font (size 1.27 1.27)) (hide yes)))
+		(property "Value" "1uF/25V" (at 139.7 219.71 0) (effects (font (size 1.27 1.27))))
+		(property "Footprint" "mp:C0402" (at 139.7 215.9 0) (effects (font (size 1.27 1.27)) (hide yes)))
+		(property "Datasheet" "https://lcsc.com/product-detail/Multilayer-Ceramic-Capacitors-MLCC-SMD-SMT_SAMSUNG_CL05A105KA5NQNC_1uF-105-10-25V_C52923.html" (at 139.7 215.9 0) (effects (font (size 1.27 1.27)) (hide yes)))
 		(property "Manufacturer" "SAMSUNG(三星)" (at 139.7 215.9 0) (effects (font (size 1.27 1.27)) (hide yes)))
-		(property "MPN" "CL10A105KB8NNNC" (at 139.7 215.9 0) (effects (font (size 1.27 1.27)) (hide yes)))
-		(property "LCSC Part" "C15849" (at 139.7 215.9 0) (effects (font (size 1.27 1.27)) (hide yes)))
-		(pin "2")
-		(pin "1")
+		(property "MPN" "CL05A105KA5NQNC" (at 139.7 215.9 0) (effects (font (size 1.27 1.27)) (hide yes)))
+		(property "LCSC Part" "C52923" (at 139.7 215.9 0) (effects (font (size 1.27 1.27)) (hide yes)))
+		(pin "1")
+		(pin "2")
 		(instances (project "mini-power" (path "/1d7b6a88-85a7-4876-8779-6fe68a207d3b" (reference "C6") (unit 1))))
 	)
@@
 	(wire (pts (xy 101.6 241.3) (xy 91.44 241.3)) (stroke (width 0) (type default)))
 	(symbol
-		(lib_id "mp:CL10A105KB8NNNC")
+		(lib_id "mp:CL05A105KA5NQNC")
 		(at 91.44 254 90)
 		(unit 1)
@@
 		(dnp no)
 		(property "Reference" "C9" (at 100.33 252.73 90) (effects (font (size 1.27 1.27))))
-		(property "Value" "1uF/50V" (at 100.33 255.27 90) (effects (font (size 1.27 1.27))))
-		(property "Footprint" "mp:C0603" (at 91.44 254 0) (effects (font (size 1.27 1.27)) (hide yes)))
-		(property "Datasheet" "https://lcsc.com/product-detail/Multilayer-Ceramic-Capacitors-MLCC-SMD-SMT_SAMSUNG_CL10A105KB8NNNC_1uF-105-10-50V_C15849.html" (at 91.44 254 0) (effects (font (size 1.27 1.27)) (hide yes)))
+		(property "Value" "1uF/25V" (at 100.33 255.27 90) (effects (font (size 1.27 1.27))))
+		(property "Footprint" "mp:C0402" (at 91.44 254 0) (effects (font (size 1.27 1.27)) (hide yes)))
+		(property "Datasheet" "https://lcsc.com/product-detail/Multilayer-Ceramic-Capacitors-MLCC-SMD-SMT_SAMSUNG_CL05A105KA5NQNC_1uF-105-10-25V_C52923.html" (at 91.44 254 0) (effects (font (size 1.27 1.27)) (hide yes)))
 		(property "Manufacturer" "SAMSUNG(三星)" (at 91.44 254 0) (effects (font (size 1.27 1.27)) (hide yes)))
-		(property "MPN" "CL10A105KB8NNNC" (at 91.44 254 0) (effects (font (size 1.27 1.27)) (hide yes)))
-		(property "LCSC Part" "C15849" (at 91.44 254 0) (effects (font (size 1.27 1.27)) (hide yes)))
-		(pin "2")
-		(pin "1")
+		(property "MPN" "CL05A105KA5NQNC" (at 91.44 254 0) (effects (font (size 1.27 1.27)) (hide yes)))
+		(property "LCSC Part" "C52923" (at 91.44 254 0) (effects (font (size 1.27 1.27)) (hide yes)))
+		(pin "1")
+		(pin "2")
 		(instances (project "mini-power" (path "/1d7b6a88-85a7-4876-8779-6fe68a207d3b" (reference "C9") (unit 1))))
 	)
@@
 	(label "A_DRV" (at 391.16 129.54 0) (effects (font (size 1.27 1.27)) (justify left bottom)))
 	(symbol
-		(lib_id "mp:CL10A105KB8NNNC")
+		(lib_id "mp:CL05A105KA5NQNC")
 		(at 416.56 129.54 0)
 		(unit 1)
@@
 		(dnp no)
 		(property "Reference" "C11" (at 416.56 125.73 0) (effects (font (size 1.27 1.27))))
-		(property "Value" "1uF/50V" (at 416.56 133.35 0) (effects (font (size 1.27 1.27))))
-		(property "Footprint" "mp:C0603" (at 416.56 129.54 0) (effects (font (size 1.27 1.27)) (hide yes)))
-		(property "Datasheet" "https://lcsc.com/product-detail/Multilayer-Ceramic-Capacitors-MLCC-SMD-SMT_SAMSUNG_CL10A105KB8NNNC_1uF-105-10-50V_C15849.html" (at 416.56 129.54 0) (effects (font (size 1.27 1.27)) (hide yes)))
+		(property "Value" "1uF/25V" (at 416.56 133.35 0) (effects (font (size 1.27 1.27))))
+		(property "Footprint" "mp:C0402" (at 416.56 129.54 0) (effects (font (size 1.27 1.27)) (hide yes)))
+		(property "Datasheet" "https://lcsc.com/product-detail/Multilayer-Ceramic-Capacitors-MLCC-SMD-SMT_SAMSUNG_CL05A105KA5NQNC_1uF-105-10-25V_C52923.html" (at 416.56 129.54 0) (effects (font (size 1.27 1.27)) (hide yes)))
 		(property "Manufacturer" "SAMSUNG(三星)" (at 416.56 129.54 0) (effects (font (size 1.27 1.27)) (hide yes)))
-		(property "MPN" "CL10A105KB8NNNC" (at 416.56 129.54 0) (effects (font (size 1.27 1.27)) (hide yes)))
-		(property "LCSC Part" "C15849" (at 416.56 129.54 0) (effects (font (size 1.27 1.27)) (hide yes)))
-		(pin "2")
-		(pin "1")
+		(property "MPN" "CL05A105KA5NQNC" (at 416.56 129.54 0) (effects (font (size 1.27 1.27)) (hide yes)))
+		(property "LCSC Part" "C52923" (at 416.56 129.54 0) (effects (font (size 1.27 1.27)) (hide yes)))
+		(pin "1")
+		(pin "2")
 		(instances (project "mini-power" (path "/1d7b6a88-85a7-4876-8779-6fe68a207d3b" (reference "C11") (unit 1))))
 	)
