File: mini-power/mini-power.kicad_pcb (KiCad board)
At the start: 2 copper layers, 100 x 100 mm, 77 parts, among them J1 Power in, J2 Power out, J3 +2.75 V in, J4 Controller rails out, J5 Controller, Q1 Si2301CDS, U1 TPS62840DLC, U2 TPS62841DLC, U3 LT8330, U4 LPV521

Commit message: Corrected PCB layout
Parts:
- C11, C6, C9: value 1uF/50V -> 1uF/25V; footprint mp:C0603 -> mp:C0402
- moved C15 31.4 mm to (175.4, 113.1)
- moved TP27 26.4 mm to (173.7, 115.1)
- moved R7 24.5 mm to (175.4, 114.5)
- moved L4 18.0 mm to (123.2, 131.6)
- moved C7 17.5 mm to (126.0, 131.1), turned to -90 degrees
- moved TP28 17.1 mm to (177.2, 117.5)
- moved U4 16.7 mm to (175.2, 116.5), turned to 90 degrees
- moved C14 16.2 mm to (175.2, 118.6), turned to 180 degrees
- moved TP10 16.0 mm to (120.2, 132.2)
- moved R6 15.0 mm to (171.9, 115.6)
- moved C6 14.5 mm to (118.5, 131.4)
- moved C2 13.6 mm to (112.3, 59.0), turned to 180 degrees
- moved L3 13.5 mm to (115.4, 131.4)
- moved C4 13.2 mm to (112.7, 85.2), turned to 180 degrees
- moved TP26 13.0 mm to (171.0, 114.6)
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Routing:
- net GND: track 3.80 -> 32.3 mm, vias 27 -> 24
- net /+3V3: track 101.4 -> 123.5 mm
- net /+2V75: track 111.1 -> 92.1 mm
- net /SNS_IN: track 22.5 -> 5.60 mm
- net /+1V4: track 32.2 -> 15.4 mm
- net /FBX_C: track 31.3 -> 18.1 mm
- net /SW_PB: track 18.2 -> 6.85 mm, vias 2 -> 0
- net /-2V75_B: track 31.4 -> 21.4 mm, vias 2 -> 0
- net /SW_C: track 15.4 -> 6.14 mm
- net /B_DRV: track 75.0 -> 66.3 mm, vias 4 -> 1
- net /A_DRV: track 41.3 -> 32.6 mm, vias 0 -> 1
- net /SENSE: track 96.1 -> 104.4 mm, vias 2 -> 0
- net /+2V8: track 25.8 -> 18.0 mm
- net /-2V8_IC: track 38.7 -> 31.0 mm
- net /N_A: track 12.7 -> 5.30 mm
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